File: board/dome-board4.sch (EAGLE design)
At the start: 13 parts

Commit message: Dome board Rev4
Parts:
- removed USB1, USB2, USB3, USB4, USB5, USB6, USB7, USB8: USB, MaxHenstell:USB
- added U$1, U$2, U$3, U$4, U$5, U$6, U$7, U$8: M04, blinkinlabs:M04
Connections:
- net GND: now also U$1.P$1, U$2.P$1, U$3.P$1, U$4.P$1, U$5.P$1, U$6.P$1, U$7.P$1, U$8.P$1, _1._GND1; no longer USB1.GND, USB2.GND, USB3.GND, USB4.GND, USB5.GND, USB6.GND, USB7.GND, USB8.GND
- net N$1: now also U$1.P$2; no longer USB1.D+
- net N$10: now also U$2.P$3; no longer USB2.D-
- net N$11: now also U$3.P$3; no longer USB3.D-
- net N$12: now also U$4.P$3; no longer USB4.D-
- net N$13: now also U$8.P$3; no longer USB5.D-
- net N$14: now also U$7.P$3; no longer USB6.D-
- net N$15: now also U$6.P$3; no longer USB7.D-
- net N$16: now also U$5.P$3; no longer USB8.D-
- net N$2: now also U$2.P$2; no longer USB2.D+
- net N$20: now also U$5.P$2; no longer USB8.D+
- net N$3: now also U$3.P$2; no longer USB3.D+
- net N$4: now also U$4.P$2; no longer USB4.D+
- net N$5: now also U$8.P$2; no longer USB5.D+
- net N$6: now also U$7.P$2; no longer USB6.D+
- net N$7: now also U$6.P$2; no longer USB7.D+
- net N$9: now also U$1.P$3; no longer USB1.D-
- net VCC1: now also U$1.P$4, U$2.P$4; no longer USB1.VBUS, USB2.VBUS
- net VCC2: now also U$5.P$4, U$6.P$4; no longer USB7.VBUS, USB8.VBUS
- net VCC3: now also U$3.P$4, U$4.P$4; no longer USB3.VBUS, USB4.VBUS
- net VCC4: now also U$7.P$4, U$8.P$4; no longer USB5.VBUS, USB6.VBUS
